Commit message: Orient the hub in the default orientation w/ USB charging port forward (+X), buttons & lights up (+Z)

File: lego_spike_description/urdf/lego_hub.urdf.xacro (robot description, xacro)
@@ -9,11 +9,11 @@
         </geometry>
         <material name="lego_white" />
-        <origin xyz="0 0 0" rpy="1.5707963267948966 0 0" />
+        <origin xyz="0.004 00.004 0" rpy="1.5707963267948966 0 -1.5707963267948966" />
       </visual>
       <collision>
         <geometry>
-          <box size="0.056 0.088 0.032" />
+          <box size="0.088 0.056 0.032" />
         </geometry>
-        <origin xyz="0.004 -0.005 0.016" rpy="0 0 0" />
+        <origin xyz="0 0 0.016" rpy="0 0 0" />
       </collision>
     </link>

Commit message: Fix the joint_state_publisher so the motors have the correct orientation; lego and ROS spin in opposite directions. Add a basic URDF with all the motors from the base kit + sensors for debugging in Rviz.

File: lego_spike_description/urdf/lego_hub.urdf.xacro (robot description, xacro)
@@ -28,5 +28,5 @@
       <child link="${name}_imu_link" />
       <!-- TODO: exact IMU position -->
-      <origin xyz="0 0 0" rpy="0 0 0" />
+      <origin xyz="0 0 0" rpy="0 0 1.57079" />
     </joint>
   </xacro:macro>

File: lego_spike_description/urdf/lego_materials.urdf.xacro (robot description, xacro)
@@ -4,3 +4,6 @@
     <color rgba="0.9 0.9 0.9 1.0" />
   </material>
+  <material name="lego_teal">
+    <color rgba="0.0 0.8 0.8 1.0" />
+  </material>
 </robot>
