Commit message: Convert the DAEs to STLs. The scale seems to have gotten mangled in the process, but I'll fix that later. Add the collision geometry for the Hub. Use a slightly off-white material to make the models show up in rviz better

File: lego_spike_description/urdf/lego_color_sensor.urdf.xacro (robot description, xacro)
@@ -5,6 +5,7 @@
       <visual>
         <geometry>
-          <mesh filename="package://lego_spike_description/meshes/SpikePrimeColorSensor.dae" scale="0.01 0.01 0.01"/>
+          <mesh filename="package://lego_spike_description/meshes/SpikePrimeColorSensor.stl" scale="0.0004 0.0004 0.0004"/>
         </geometry>
+        <material name="lego_white" />
         <origin xyz="0 0 0" rpy="1.5707963267948966 0 1.5707963267948966" />
       </visual>

File: lego_spike_description/urdf/lego_distance_sensor.urdf.xacro (robot description, xacro)
@@ -5,6 +5,7 @@
       <visual>
         <geometry>
-          <mesh filename="package://lego_spike_description/meshes/SpikePrimeDistanceSensor.dae" scale="0.01 0.01 0.01"/>
+          <mesh filename="package://lego_spike_description/meshes/SpikePrimeDistanceSensor.stl" scale="0.0004 0.0004 0.0004"/>
         </geometry>
+        <material name="lego_white" />
         <origin xyz="0 0 0" rpy="1.5707963267948966 0 1.5707963267948966" />
       </visual>

File: lego_spike_description/urdf/lego_force_sensor.urdf.xacro (robot description, xacro)
@@ -5,6 +5,7 @@
       <visual>
         <geometry>
-          <mesh filename="package://lego_spike_description/meshes/SpikePrimeForceSensor.dae" scale="0.01 0.01 0.01"/>
+          <mesh filename="package://lego_spike_description/meshes/SpikePrimeForceSensor.stl" scale="0.0004 0.0004 0.0004"/>
         </geometry>
+        <material name="lego_white" />
         <origin xyz="0 0 0" rpy="1.5707963267948966 0 1.5707963267948966" />
       </visual>

File: lego_spike_description/urdf/lego_hub.urdf.xacro (robot description, xacro)
@@ -1,13 +1,20 @@
 <?xml version="1.0" ?>
 <robot xmlns:xacro="http://wiki.ros.org/xacro">
+  <xacro:include filename="$(find lego_spike_description)/urdf/lego_materials.urdf.xacro" />
   <xacro:macro name="lego_hub" params="name parent *origin">
     <link name="${name}_link">
       <visual>
         <geometry>
-          <mesh filename="package://lego_spike_description/meshes/SpikePrimeHub.dae" scale="0.01 0.01 0.01"/>
+          <mesh filename="package://lego_spike_description/meshes/SpikePrimeHub.stl" scale="0.0004 0.0004 0.0004"/>
         </geometry>
+        <material name="lego_white" />
         <origin xyz="0 0 0" rpy="1.5707963267948966 0 0" />
       </visual>
-      <!-- TODO: collision -->
+      <collision>
+        <geometry>
+          <box size="0.056 0.088 0.032" />
+        </geometry>
+        <origin xyz="0.004 -0.005 0.016" rpy="0 0 0" />
+      </collision>
     </link>
     <joint name="${name}_joint" type="fixed">

File: lego_spike_description/urdf/lego_large_motor.urdf.xacro (robot description, xacro)
@@ -5,6 +5,7 @@
       <visual>
         <geometry>
-          <mesh filename="package://lego_spike_description/meshes/SpikePrimeLargeMotor.dae" scale="0.01 0.01 0.01"/>
+          <mesh filename="package://lego_spike_description/meshes/SpikePrimeLargeMotor.stl" scale="0.0004 0.0004 0.0004"/>
         </geometry>
+        <material name="lego_white" />
         <origin xyz="0 0.005 0" rpy="1.5707963267948966 0 1.5707963267948966" />
       </visual>

File: lego_spike_description/urdf/lego_materials.urdf.xacro (robot description, xacro)
@@ -2,5 +2,5 @@
 <robot xmlns:xacro="http://wiki.ros.org/xacro">
   <material name="lego_white">
-    <color rgba="0.8 0.8 0.8 1.0" />
+    <color rgba="0.9 0.9 0.9 1.0" />
   </material>
 </robot>

File: lego_spike_description/urdf/lego_small_motor.urdf.xacro (robot description, xacro)
@@ -5,6 +5,7 @@
       <visual>
         <geometry>
-          <mesh filename="package://lego_spike_description/meshes/SpikePrimeSmallMotor.dae" scale="0.01 0.01 0.01"/>
+          <mesh filename="package://lego_spike_description/meshes/SpikePrimeSmallMotor.stl" scale="0.0004 0.0004 0.0004"/>
         </geometry>
+        <material name="lego_white" />
         <origin xyz="0 0.005 0" rpy="1.5707963267948966 0 1.5707963267948966" />
       </visual>

Commit message: Restrict the names of of the lego sensors and motors to be associated with the ports they're connected to. Publish the distance sensor data as an array of point clouds. Remove the testing description to add the accessories to a Jackal

File: lego_spike_description/urdf/lego_color_sensor.urdf.xacro (robot description, xacro)
@@ -1,6 +1,6 @@
 <?xml version="1.0" ?>
 <robot xmlns:xacro="http://wiki.ros.org/xacro">
-  <xacro:macro name="lego_color_sensor" params="name parent *origin">
-    <link name="${name}_link">
+  <xacro:macro name="lego_color_sensor" params="port parent *origin">
+    <link name="color_${port}_link">
       <visual>
         <geometry>
@@ -12,7 +12,7 @@
       <!-- TODO: collision -->
     </link>
-    <joint name="${name}_joint" type="fixed">
+    <joint name="color_${port}_joint" type="fixed">
       <parent link="${parent}" />
-      <child link="${name}_link" />
+      <child link="color_${port}_link" />
       <xacro:insert_block name="origin" />
     </joint>

File: lego_spike_description/urdf/lego_distance_sensor.urdf.xacro (robot description, xacro)
@@ -1,6 +1,6 @@
 <?xml version="1.0" ?>
 <robot xmlns:xacro="http://wiki.ros.org/xacro">
-  <xacro:macro name="lego_distance_sensor" params="name parent *origin">
-    <link name="${name}_link">
+  <xacro:macro name="lego_distance_sensor" params="port parent *origin">
+    <link name="distance_${port}_link">
       <visual>
         <geometry>
@@ -12,7 +12,7 @@
       <!-- TODO: collision -->
     </link>
-    <joint name="${name}_joint" type="fixed">
+    <joint name="distance_${port}_joint" type="fixed">
       <parent link="${parent}" />
-      <child link="${name}_link" />
+      <child link="distance_${port}_link" />
       <xacro:insert_block name="origin" />
     </joint>

File: lego_spike_description/urdf/lego_force_sensor.urdf.xacro (robot description, xacro)
@@ -1,6 +1,6 @@
 <?xml version="1.0" ?>
 <robot xmlns:xacro="http://wiki.ros.org/xacro">
-  <xacro:macro name="lego_force_sensor" params="name parent *origin">
-    <link name="${name}_link">
+  <xacro:macro name="lego_force_sensor" params="port parent *origin">
+    <link name="force_${port}_link">
       <visual>
         <geometry>
@@ -12,7 +12,7 @@
       <!-- TODO: collision -->
     </link>
-    <joint name="${name}_joint" type="fixed">
+    <joint name="force_${port}_joint" type="fixed">
       <parent link="${parent}" />
-      <child link="${name}_link" />
+      <child link="force_${port}_link" />
       <xacro:insert_block name="origin" />
     </joint>

File: lego_spike_description/urdf/lego_large_motor.urdf.xacro (robot description, xacro)
@@ -1,6 +1,6 @@
 <?xml version="1.0" ?>
 <robot xmlns:xacro="http://wiki.ros.org/xacro">
-  <xacro:macro name="lego_large_motor" params="name parent *origin">
-    <link name="${name}_link">
+  <xacro:macro name="lego_large_motor" params="port parent *origin">
+    <link name="motor_${port}_link">
       <visual>
         <geometry>
@@ -12,13 +12,13 @@
       <!-- TODO: collision -->
     </link>
-    <joint name="${name}_joint" type="fixed">
+    <joint name="motor_${port}_joint" type="fixed">
       <parent link="${parent}" />
-      <child link="${name}_link" />
+      <child link="motor_${port}_link" />
       <xacro:insert_block name="origin" />
     </joint>
-    <link name="${name}_wheel_link" />
-    <joint name="${name}_wheel_joint" type="continuous">
-      <parent link="${name}_link" />
-      <child link="${name}_wheel_link" />
+    <link name="motor_${port}_wheel_link" />
+    <joint name="motor_${port}_wheel_joint" type="continuous">
+      <parent link="motor_${port}_link" />
+      <child link="motor_${port}_wheel_link" />
       <origin xyz="0.02 0 0.03" rpy="0 0 0" />
       <axis xyz="0 0 1" />

File: lego_spike_description/urdf/lego_robot.urdf.xacro (robot description, xacro)
@@ -13,20 +13,20 @@
     <origin xyz="0.1 0 0" rpy="0 0 0" />
   </xacro:lego_hub>
-  <xacro:lego_small_motor name="motor_a" parent="base_link">
+  <xacro:lego_small_motor port="a" parent="base_link">
     <origin xyz="0 0.032 0.008" rpy="0 0 3.14150" />
   </xacro:lego_small_motor>
-  <xacro:lego_small_motor name="motor_b" parent="base_link">
+  <xacro:lego_small_motor port="b" parent="base_link">
     <origin xyz="0 -0.064 0.008" rpy="0 0 3.14150" />
   </xacro:lego_small_motor>
-  <xacro:lego_small_motor name="motor_c" parent="base_link">
+  <xacro:lego_small_motor port="c" parent="base_link">
     <origin xyz="0 0 0.008" rpy="0 0 3.14150" />
   </xacro:lego_small_motor>
-  <xacro:lego_small_motor name="motor_d" parent="base_link">
+  <xacro:lego_small_motor port="d" parent="base_link">
     <origin xyz="0 -0.032 0.008" rpy="0 0 3.14150" />
   </xacro:lego_small_motor>
-  <xacro:lego_distance_sensor name="distance_e" parent="base_link">
+  <xacro:lego_distance_sensor port="e" parent="base_link">
     <origin xyz="-0.016 0.054 0.038" rpy="1.57079 0 3.14150" />
   </xacro:lego_distance_sensor>
-  <xacro:lego_color_sensor name="color_f" parent="motor_b_wheel_link">
+  <xacro:lego_color_sensor port="f" parent="motor_b_wheel_link">
     <origin xyz="0 0 0" rpy="0 0 0" />
   </xacro:lego_color_sensor>

File: lego_spike_description/urdf/lego_small_motor.urdf.xacro (robot description, xacro)
@@ -1,6 +1,6 @@
 <?xml version="1.0" ?>
 <robot xmlns:xacro="http://wiki.ros.org/xacro">
-  <xacro:macro name="lego_small_motor" params="name parent *origin">
-    <link name="${name}_link">
+  <xacro:macro name="lego_small_motor" params="port parent *origin">
+    <link name="motor_${port}_link">
       <visual>
         <geometry>
@@ -12,13 +12,13 @@
       <!-- TODO: collision -->
     </link>
-    <joint name="${name}_joint" type="fixed">
+    <joint name="motor_${port}_joint" type="fixed">
       <parent link="${parent}" />
-      <child link="${name}_link" />
+      <child link="motor_${port}_link" />
       <xacro:insert_block name="origin" />
     </joint>
-    <link name="${name}_wheel_link" />
-    <joint name="${name}_wheel_joint" type="continuous">
-      <parent link="${name}_link" />
-      <child link="${name}_wheel_link" />
+    <link name="motor_${port}_wheel_link" />
+    <joint name="motor_${port}_wheel_joint" type="continuous">
+      <parent link="motor_${port}_link" />
+      <child link="motor_${port}_wheel_link" />
       <origin xyz="0.02 0 0.03" rpy="0 0 0" />
       <axis xyz="0 0 1" />
