Commit message: Refactor all of the sensors/motors so their links align with the actual lego. Define properties corresponding to lego piece dimensions to make building URDFs that align with Lego easier. Remove the large motor as I don't have one to test with. Rename small motor to just motor, as it turns out there's a third, even-smaller motor.

File: lego_spike_description/urdf/lego_base_plate.urdf.xacro (robot description, xacro)
@@ -1,4 +1,9 @@
 <?xml version="1.0" ?>
 <robot xmlns:xacro="http://wiki.ros.org/xacro">
+  <xacro:include filename="$(find lego_spike_description)/urdf/lego_dimensions.urdf.xacro" />
+  <!--
+    The 11x19 hole lego technic plate included in Lego Mindstorms 51515
+    Model is centered on the middle with the long dimension along the X axis
+  -->
   <xacro:macro name="lego_base_plate" params="name parent *origin">
     <link name="${name}_link">
@@ -8,5 +13,5 @@
         </geometry>
         <material name="lego_teal" />
-        <origin xyz="0.004 00.004 0" rpy="1.5707963267948966 0 -1.5707963267948966" />
+        <origin xyz="-${lego_stud_spacing*1.5} -${lego_stud_spacing/2} 0" rpy="1.5707963267948966 0 -1.5707963267948966" />
       </visual>
     </link>
@@ -16,4 +21,11 @@
       <xacro:insert_block name="origin" />
     </joint>
+    <link name="${name}_top_link" />
+    <joint name="${name}_top_joint" type="fixed">
+      <parent link="${name}_link" />
+      <child link="${name}_top_link" />
+      <!-- Height is the width of a standard brick, not the height of a brick! -->
+      <origin xyz="0 0 ${lego_brick_width}" rpy="0 0 0" />
+    </joint>
   </xacro:macro>
 </robot>

File: lego_spike_description/urdf/lego_color_sensor.urdf.xacro (robot description, xacro)
@@ -1,4 +1,9 @@
 <?xml version="1.0" ?>
 <robot xmlns:xacro="http://wiki.ros.org/xacro">
+  <xacro:include filename="$(find lego_spike_description)/urdf/lego_dimensions.urdf.xacro" />
+  <!--
+    Lego Mindstorms 51515 color/light sensor.
+    Origin is the center-back near the cable attachment, rounded edges up/down
+  -->
   <xacro:macro name="lego_color_sensor" params="port parent *origin">
     <link name="color_${port}_link">
@@ -8,5 +13,5 @@
         </geometry>
         <material name="lego_white" />
-        <origin xyz="0 0 0" rpy="1.5707963267948966 0 1.5707963267948966" />
+        <origin xyz="${lego_stud_spacing} 0 -${lego_stud_spacing * 1.5}" rpy="1.5707963267948966 0 1.5707963267948966" />
       </visual>
       <!-- TODO: collision -->

File: lego_spike_description/urdf/lego_distance_sensor.urdf.xacro (robot description, xacro)
@@ -1,4 +1,10 @@
 <?xml version="1.0" ?>
 <robot xmlns:xacro="http://wiki.ros.org/xacro">
+  <xacro:include filename="$(find lego_spike_description)/urdf/lego_dimensions.urdf.xacro" />
+  <!--
+    Lego Mindstorms 51515 ultrasonic range sensor
+    Origin is the center-back, near the cable connection. Emitter & receiver point forward along the X axis.
+    Measurements relative to the origin of the model.
+  -->
   <xacro:macro name="lego_distance_sensor" params="port parent *origin">
     <link name="distance_${port}_link">
@@ -8,5 +14,5 @@
         </geometry>
         <material name="lego_white" />
-        <origin xyz="0 0 0" rpy="1.5707963267948966 0 1.5707963267948966" />
+        <origin xyz="${lego_stud_spacing * 1.5} 0 -${lego_stud_spacing * 1.5}" rpy="1.5707963267948966 0 1.5707963267948966" />
       </visual>
       <!-- TODO: collision -->

File: lego_spike_description/urdf/lego_force_sensor.urdf.xacro (robot description, xacro)
@@ -1,4 +1,5 @@
 <?xml version="1.0" ?>
 <robot xmlns:xacro="http://wiki.ros.org/xacro">
+  <xacro:include filename="$(find lego_spike_description)/urdf/lego_dimensions.urdf.xacro" />
   <xacro:macro name="lego_force_sensor" params="port parent *origin">
     <link name="force_${port}_link">

File: lego_spike_description/urdf/lego_hub.urdf.xacro (robot description, xacro)
@@ -1,5 +1,5 @@
 <?xml version="1.0" ?>
 <robot xmlns:xacro="http://wiki.ros.org/xacro">
-  <xacro:include filename="$(find lego_spike_description)/urdf/lego_materials.urdf.xacro" />
+  <xacro:include filename="$(find lego_spike_description)/urdf/lego_dimensions.urdf.xacro" />
   <xacro:macro name="lego_hub" params="name parent *origin">
     <link name="${name}_link">

File: lego_spike_description/urdf/lego_materials.urdf.xacro (robot description, xacro)
@@ -7,3 +7,6 @@
     <color rgba="0.0 0.8 0.8 1.0" />
   </material>
+  <material name="lego_yellow">
+    <color rgba="0.8 0.8 0.0 1.0" />
+  </material>
 </robot>
