Commit message: Add collision boxes to the motors & sensor. Remove the force sensor (because I don't have one to test with). Move the .rviz config into the package, add the env_runner scripts, update the description cmake. Start adding the arm URDF. Need to finish designing in stud.io and exporting the meshes before I can finish that up.

File: lego_spike_description/urdf/basic_lego_robot.urdf.xacro (robot description, xacro)
@@ -1,4 +1,4 @@
 <?xml version="1.0" ?>
-<robot name="lego_mindstorms" xmlns:xacro="http://wiki.ros.org/xacro">
+<robot name="basic_robot" xmlns:xacro="http://wiki.ros.org/xacro">
   <xacro:include filename="$(find lego_spike_description)/urdf/lego_materials.urdf.xacro" />
   <xacro:include filename="$(find lego_spike_description)/urdf/lego_hub.urdf.xacro" />

File: lego_spike_description/urdf/lego_arm.urdf.xacro (robot description, xacro)
@@ -1,3 +1,16 @@
 <?xml version="1.0" ?>
 <robot name="lego_arm" xmlns:xacro="http://wiki.ros.org/xacro">
+  <xacro:include filename="$(find lego_spike_description)/urdf/lego_materials.urdf.xacro" />
+  <xacro:include filename="$(find lego_spike_description)/urdf/lego_hub.urdf.xacro" />
+  <xacro:include filename="$(find lego_spike_description)/urdf/lego_base_plate.urdf.xacro" />
+  <xacro:include filename="$(find lego_spike_description)/urdf/lego_motor.urdf.xacro" />
+  <xacro:include filename="$(find lego_spike_description)/urdf/lego_distance_sensor.urdf.xacro" />
+  <xacro:include filename="$(find lego_spike_description)/urdf/lego_color_sensor.urdf.xacro" />
+  <link name="base_link" />
+  <xacro:lego_base_plate name="base_plate" parent="base_link">
+    <origin xyz="0 0 0" rpy="0 0 1.57079" />
+  </xacro:lego_base_plate>
+  <xacro:lego_hub name="lego_hub" parent="base_plate_top_link">
+    <origin xyz="-${lego_stud_spacing * 6} 0 0" rpy="0 0 -${pi/2}" />
+  </xacro:lego_hub>
 </robot>

File: lego_spike_description/urdf/lego_base_plate.urdf.xacro (robot description, xacro)
@@ -15,4 +15,10 @@
         <origin xyz="-${lego_stud_spacing*1.5} -${lego_stud_spacing/2} 0" rpy="1.5707963267948966 0 -1.5707963267948966" />
       </visual>
+      <collision>
+        <geometry>
+          <box size="${lego_stud_spacing * 19} ${lego_stud_spacing * 11} ${lego_stud_spacing}" />
+        </geometry>
+        <origin xyz="0 0 ${lego_brick_width/2}" rpy="0 0 0" />
+      </collision>
     </link>
     <joint name="${name}_joint" type="fixed">

File: lego_spike_description/urdf/lego_color_sensor.urdf.xacro (robot description, xacro)
@@ -15,5 +15,10 @@
         <origin xyz="${lego_stud_spacing} 0 -${lego_stud_spacing * 1.5}" rpy="1.5707963267948966 0 1.5707963267948966" />
       </visual>
-      <!-- TODO: collision -->
+      <collision>
+        <geometry>
+          <box size="${lego_stud_spacing * 3} ${lego_stud_spacing * 3} ${lego_stud_spacing * 3}" />
+        </geometry>
+        <origin xyz="${lego_stud_spacing * 1} 0 0" rpy="0 0 0" />
+      </collision>
     </link>
     <joint name="color_${port}_joint" type="fixed">

File: lego_spike_description/urdf/lego_distance_sensor.urdf.xacro (robot description, xacro)
@@ -16,5 +16,10 @@
         <origin xyz="${lego_stud_spacing * 1.5} 0 -${lego_stud_spacing * 1.5}" rpy="1.5707963267948966 0 1.5707963267948966" />
       </visual>
-      <!-- TODO: collision -->
+      <collision>
+        <geometry>
+          <box size="${lego_stud_spacing * 4} ${lego_stud_spacing * 7} ${lego_stud_spacing * 3}" />
+        </geometry>
+        <origin xyz="${lego_stud_spacing * 1.5} 0 0" rpy="0 0 0" />
+      </collision>
     </link>
     <joint name="distance_${port}_joint" type="fixed">

File: lego_spike_description/urdf/lego_motor.urdf.xacro (robot description, xacro)
@@ -15,5 +15,10 @@
         <origin xyz="${lego_stud_spacing/2} 0.0045 0" rpy="1.5707963267948966 0 1.5707963267948966" />
       </visual>
-      <!-- TODO: collision -->
+      <collision>
+        <geometry>
+          <box size="${lego_stud_spacing * 9} ${lego_stud_spacing * 3} ${lego_stud_spacing * 3}" />
+        </geometry>
+        <origin xyz="0 0 ${lego_stud_spacing * 1.5}" rpy="0 0 0" />
+      </collision>
     </link>
     <joint name="motor_${port}_joint" type="fixed">
@@ -22,5 +27,12 @@
       <xacro:insert_block name="origin" />
     </joint>
-    <link name="motor_${port}_wheel_link" />
+    <link name="motor_${port}_wheel_link">
+      <collision>
+        <geometry>
+          <cylinder radius="${lego_stud_spacing * 1.5}" length="${lego_stud_spacing}" />
+        </geometry>
+        <origin xyz="0 0 -${lego_stud_spacing * 0.5}" rpy="0 0 0" />
+      </collision>
+    </link>
     <joint name="motor_${port}_wheel_joint" type="continuous">
       <parent link="motor_${port}_link" />
