Commit message: Add a simple robot arm with building instructions, static elements exported from Stud.io

File: lego_spike_description/urdf/lego_materials.urdf.xacro (robot description, xacro)
@@ -3,4 +3,7 @@
   <material name="lego_white">
     <color rgba="0.9 0.9 0.9 1.0" />
+  </material>
+  <material name="lego_black">
+    <color rgba="0.1 0.1 0.1 1.0" />
   </material>
   <material name="lego_teal">
