Commit message: Redesign the arm slightly with a better gripper

File: lego_spike_description/urdf/simple_arm.urdf.xacro (robot description, xacro)
@@ -13,5 +13,5 @@
   </xacro:lego_base_plate>
   <xacro:lego_hub name="lego_hub" parent="base_plate_top_link">
-    <origin xyz="-${lego_stud_spacing * 6} 0 0" rpy="0 0 -${pi/2}" />
+    <origin xyz="-${lego_stud_spacing * 6} 0 ${lego_stud_spacing * 1}" rpy="0 0 -${pi/2}" />
   </xacro:lego_hub>
   <xacro:lego_motor port="b" parent="base_plate_top_link">
@@ -99,5 +99,5 @@
       </geometry>
       <material name="lego_black" />
-      <origin xyz="${lego_stud_spacing * 0.5} ${lego_stud_spacing * 2.5} -${lego_stud_spacing * 2}" rpy="${pi/2} -${pi/2} ${pi/2}" />
+      <origin xyz="-${lego_stud_spacing * 3} ${lego_stud_spacing * 4.5} -${lego_stud_spacing * 1.5}" rpy="${pi/2} -${pi/2} ${pi/2}" />
     </visual>
     <collision>
@@ -105,5 +105,5 @@
         <mesh filename="package://lego_spike_description/meshes/mobile_fingers.stl" scale="0.0004 0.0004 0.0004"/>
       </geometry>
-      <origin xyz="${lego_stud_spacing * 0.5} ${lego_stud_spacing * 2.5} -${lego_stud_spacing * 2}" rpy="${pi/2} -${pi/2} ${pi/2}" />
+      <origin xyz="-${lego_stud_spacing * 3} ${lego_stud_spacing * 4.5} -${lego_stud_spacing * 1.5}" rpy="${pi/2} -${pi/2} ${pi/2}" />
     </collision>
   </link>
